File: board/coffeere.brd (EAGLE design)
At the start: 100 x 50 mm, 17 parts, among them J1 STATUS LED

Commit message: Fixing board issues
Parts:
- moved U$1 6.35 mm to (31.5, 43.1)
- moved SV2 6.00 mm to (56.5, 24.6)
- moved J1 4.12 mm to (48.5, 14.9)
- moved R2 4.12 mm to (45.0, 6.90)
- moved C2 3.16 mm to (51.6, 44.9)
- moved R1 2.24 mm to (45.4, 28.6)
- moved CN2 2.00 mm to (12.0, 47.0)
- moved J3 2.00 mm to (23.6, 16.9), turned to 180 degrees
- moved AMS1117 1.00 mm to (8.60, 25.7)
- moved SV1 1.00 mm to (28.5, 22.9)
Routing:
- net GND: track 0.00 -> 64.7 mm, vias 0 -> 6
- net GPIO2: track 15.4 -> 24.8 mm
- net 3.3V: track 153.9 -> 161.6 mm
- net GPIO13: track 24.8 -> 31.6 mm
- net N$16: track 20.8 -> 27.6 mm
- net N$13: track 9.53 -> 14.8 mm
- net N$12: track 13.0 -> 17.7 mm
- net GPIO14: track 35.4 -> 30.9 mm
- net GPIO12: track 31.3 -> 26.7 mm
- net GPIO16: track 50.7 -> 55.2 mm
- net GPIO0: track 43.4 -> 47.0 mm
- net N$17: track 13.8 -> 15.7 mm
- net GPIO15: track 7.43 -> 9.13 mm
- net GPIO4: track 23.4 -> 24.8 mm
- net N$2: track 7.09 -> 8.09 mm
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